Commit message: moveit_gazebo.launch for doosan & gripper

File: dsr_description/xacro/a0912.urdf.xacro (robot description, xacro)
@@ -3,5 +3,5 @@
   <xacro:arg name="color"   default="white"/>
   <xacro:arg name="gripper" default="none"/>
-  <xacro:arg name="ns" default="dsr"/>
+  <xacro:arg name="ns" default="dsr01"/>
   <xacro:property name="cr" value="$(arg color)"/>
   <xacro:property name="gr" value="$(arg gripper)"/>

File: dsr_description/xacro/macro.a0912.white.xacro (robot description, xacro)
@@ -6,4 +6,10 @@
 	<xacro:macro name="a0912" params="namespace">
 		<xacro:dsr_materials />
+		<!-- <link name="world">
+		<joint name="world_fix" type="fix">
+			<origin rpy="0 0 0" xyz="0 0 0"/>
+			<parent link="world"/>
+			<child link="base_0"/>
+		</joint> -->
 		<link name="base_0">
 			<inertial>
@@ -228,4 +234,10 @@
 			</visual>
 		</link>
+		<link name="tcp"/>
+		<joint name="jointtcp" type="fixed">
+			<origin rpy="0 0 0" xyz="0 0 0.185"/>
+			<parent link="link6"/>
+			<child link="tcp"/>
+		</joint>
 		<xacro:dsr_transmission />
 		<xacro:dsr_gazebo namespace="${namespace}" />

Commit message: RAI-Lab ubuntu 20.04 noetic with doosan-robot & robotiq_140_gripper test success

File: dsr_description/xacro/a0912.urdf.xacro (robot description, xacro)
@@ -3,4 +3,5 @@
   <xacro:arg name="color"   default="white"/>
   <xacro:arg name="gripper" default="none"/>
+  <xacro:arg name="ns" default="dsr01"/>
   <xacro:property name="cr" value="$(arg color)"/>
   <xacro:property name="gr" value="$(arg gripper)"/>
@@ -11,9 +12,9 @@
      <xacro:include filename="$(find dsr_description)/xacro/macro.a0912.blue.xacro" />
   </xacro:if>
-  <xacro:a0912 namespace="$(arg namespace)"/>
+  <xacro:a0912 namespace="$(arg ns)"/>
   <link name="world" />
-  <xacro:if value="${gr == 'robotiq_2f'}">
+  <!--xacro:if value="${gr == 'robotiq_2f'}">
      <xacro:include filename="$(find dsr_description)/xacro/robotiq_2f.urdf.xacro" />
-  </xacro:if>
+  </xacro:if-->
   <!-- World fixed joint-->
   <joint name="world_fixed" type="fixed">

File: dsr_description/xacro/macro.a0912.white.xacro (robot description, xacro)
@@ -6,4 +6,10 @@
 	<xacro:macro name="a0912" params="namespace">
 		<xacro:dsr_materials />
+		<!-- <link name="world">
+		<joint name="world_fix" type="fix">
+			<origin rpy="0 0 0" xyz="0 0 0"/>
+			<parent link="world"/>
+			<child link="base_0"/>
+		</joint> -->
 		<link name="base_0">
 			<inertial>
@@ -14,4 +20,9 @@
 					izz="0.021063"/>
 				</inertial>
+			<collision>
+                <geometry>
+                    <cylinder radius="0.02" length="0.001"/>
+                </geometry>
+            </collision>
 			<visual>
 				<origin rpy="0 0 0" xyz="0 0 0" />
@@ -120,4 +131,9 @@
 					izz="0.0080652"/>
 			</inertial>
+			<collision>
+                <geometry>
+                    <cylinder radius="0.02" length="0.001"/>
+                </geometry>
+            </collision>
 			<visual>
 				<origin rpy="0 0 0" xyz="0 0 0" />
@@ -221,4 +237,9 @@
 					izz="0.0059696"/>
 			</inertial>
+			<collision>
+                <geometry>
+                    <cylinder radius="0.002" length="0.0001"/>
+                </geometry>
+            </collision>
 			<visual>
 				<origin rpy="0 0 0" xyz="0 0 0" />
@@ -228,4 +249,10 @@
 			</visual>
 		</link>
+		<link name="tcp"/>
+		<joint name="jointtcp" type="fixed">
+			<origin rpy="0 0 0" xyz="0 0 0.185"/>
+			<parent link="link6"/>
+			<child link="tcp"/>
+		</joint>
 		<xacro:dsr_transmission />
 		<xacro:dsr_gazebo namespace="${namespace}" />
